File: hardware/numpad/01_power_usb.kicad_sch (KiCad schematic)
At the start: 7 parts, among them J1 USB_C_Receptacle_USB2.0_16P, U1 USBLC6-2SC6, U2 NCP1117-3.3_SOT223

Commit message: matrix sheet, encoder, root hierarchy wired
Parts:
- renumbered R2 to R1, R1 to R2, U2 to U1, U1 to U2
Changed lines of the file:
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@@
 		)
 	)
-	(label "USB_DP"
+	(hierarchical_label "USB_DM"
+		(shape input)
+		(at 168.91 106.68 0)
+		(effects
+			(font
+				(size 1.27 1.27)
+			)
+			(justify left)
+		)
+	)
+	(hierarchical_label "USB_DP"
+		(shape input)
 		(at 168.91 104.14 0)
 		(effects
@@
 				(size 1.27 1.27)
 			)
-			(justify left bottom)
-		)
-	)
-	(label "USB_DM"
-		(at 168.91 106.68 0)
-		(effects
-			(font
-				(size 1.27 1.27)
-			)
-			(justify left bottom)
+			(justify left)
 		)
 	)
@@
 		(dnp no)
 		(fields_autoplaced yes)
-		(property "Reference" "R2"
+		(property "Reference" "R1"
 			(at 129.54 91.4399 0)
 			(show_name no)
@@
 			(project "numpad"
 				(path "/a21b85ed-e0a7-4fe0-8fc3-9355226ce8a2/4e121569-762a-4ac6-b1db-df36057e61df"
-					(reference "R2")
+					(reference "R1")
 					(unit 1)
 				)
@@
 		(dnp no)
 		(fields_autoplaced yes)
-		(property "Reference" "U2"
+		(property "Reference" "U1"
 			(at 196.85 77.47 0)
 			(show_name no)
@@
 			(project "numpad"
 				(path "/a21b85ed-e0a7-4fe0-8fc3-9355226ce8a2/4e121569-762a-4ac6-b1db-df36057e61df"
-					(reference "U2")
+					(reference "U1")
 					(unit 1)
 				)
@@
 		(dnp no)
 		(fields_autoplaced yes)
-		(property "Reference" "#PWR07"
+		(property "Reference" "#PWR08"
 			(at 92.71 132.08 0)
 			(hide yes)
@@
 			(project "numpad"
 				(path "/a21b85ed-e0a7-4fe0-8fc3-9355226ce8a2/4e121569-762a-4ac6-b1db-df36057e61df"
-					(reference "#PWR07")
+					(reference "#PWR08")
 					(unit 1)
 				)
@@
 		(dnp no)
 		(fields_autoplaced yes)
-		(property "Reference" "U1"
+		(property "Reference" "U2"
 			(at 159.1311 96.52 0)
 			(show_name no)
@@
 			(project "numpad"
 				(path "/a21b85ed-e0a7-4fe0-8fc3-9355226ce8a2/4e121569-762a-4ac6-b1db-df36057e61df"
-					(reference "U1")
+					(reference "U2")
 					(unit 1)
 				)
@@
 		(dnp no)
 		(fields_autoplaced yes)
-		(property "Reference" "#PWR01"
+		(property "Reference" "#PWR02"
 			(at 148.59 86.36 0)
 			(hide yes)
@@
 			(project "numpad"
 				(path "/a21b85ed-e0a7-4fe0-8fc3-9355226ce8a2/4e121569-762a-4ac6-b1db-df36057e61df"
-					(reference "#PWR01")
+					(reference "#PWR02")
 					(unit 1)
 				)
@@
 		(dnp no)
 		(fields_autoplaced yes)
-		(property "Reference" "#PWR05"
+		(property "Reference" "#PWR07"
 			(at 157.48 120.65 0)
 			(hide yes)
@@
 			(project "numpad"
 				(path "/a21b85ed-e0a7-4fe0-8fc3-9355226ce8a2/4e121569-762a-4ac6-b1db-df36057e61df"
-					(reference "#PWR05")
+					(reference "#PWR07")
 					(unit 1)
 				)
@@
 		(dnp no)
 		(fields_autoplaced yes)
-		(property "Reference" "#PWR08"
+		(property "Reference" "#PWR03"
 			(at 182.88 97.79 0)
 			(hide yes)
@@
 			(project "numpad"
 				(path "/a21b85ed-e0a7-4fe0-8fc3-9355226ce8a2/4e121569-762a-4ac6-b1db-df36057e61df"
-					(reference "#PWR08")
+					(reference "#PWR03")
 					(unit 1)
 				)
@@
 		(dnp no)
 		(fields_autoplaced yes)
-		(property "Reference" "#PWR04"
+		(property "Reference" "#PWR01"
 			(at 214.63 80.01 0)
 			(hide yes)
@@
 			(project "numpad"
 				(path "/a21b85ed-e0a7-4fe0-8fc3-9355226ce8a2/4e121569-762a-4ac6-b1db-df36057e61df"
-					(reference "#PWR04")
+					(reference "#PWR01")
 					(unit 1)
 				)
@@
 		(dnp no)
 		(fields_autoplaced yes)
-		(property "Reference" "R1"
+		(property "Reference" "R2"
 			(at 149.86 91.4399 0)
 			(show_name no)
@@
 			(project "numpad"
 				(path "/a21b85ed-e0a7-4fe0-8fc3-9355226ce8a2/4e121569-762a-4ac6-b1db-df36057e61df"
-					(reference "R1")
+					(reference "R2")
 					(unit 1)
 				)
@@
 		(dnp no)
 		(fields_autoplaced yes)
-		(property "Reference" "#PWR03"
+		(property "Reference" "#PWR04"
 			(at 196.85 97.79 0)
 			(hide yes)
@@
 			(project "numpad"
 				(path "/a21b85ed-e0a7-4fe0-8fc3-9355226ce8a2/4e121569-762a-4ac6-b1db-df36057e61df"
-					(reference "#PWR03")
+					(reference "#PWR04")
 					(unit 1)
 				)
@@
 		(dnp no)
 		(fields_autoplaced yes)
-		(property "Reference" "#PWR09"
+		(property "Reference" "#PWR05"
 			(at 209.55 97.79 0)
 			(hide yes)
@@
 			(project "numpad"
 				(path "/a21b85ed-e0a7-4fe0-8fc3-9355226ce8a2/4e121569-762a-4ac6-b1db-df36057e61df"
-					(reference "#PWR09")
-					(unit 1)
-				)
+					(reference "#PWR05")
+					(unit 1)
+				)

Commit message: Format cleanup, titles
Other:
- title: (none) -> Power and USB-C
- moved on the sheet: C1, C2, J1, R1, R2, U1, U2

Commit message: footprints set
Parts:
- C1, C2: footprint (none) -> Capacitor_SMD:C_0805_2012Metric
- J1: footprint (none) -> Connector_USB:USB_C_Receptacle_HRO_TYPE-C-31-M-12
- R1, R2: footprint (none) -> Resistor_SMD:R_0603_1608Metric
Changed lines of the file:
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@@
 			)
 		)
-		(property "Footprint" ""
+		(property "Footprint" "Resistor_SMD:R_0603_1608Metric"
 			(at 80.772 59.69 90)
 			(hide yes)
@@
 			)
 		)
-		(property "Footprint" ""
+		(property "Footprint" "Capacitor_SMD:C_0805_2012Metric"
 			(at 167.3352 55.88 0)
 			(hide yes)
@@
 			)
 		)
-		(property "Footprint" ""
+		(property "Footprint" "Resistor_SMD:R_0603_1608Metric"
 			(at 101.092 59.69 90)
 			(hide yes)
@@
 			)
 		)
-		(property "Footprint" ""
+		(property "Footprint" "Connector_USB:USB_C_Receptacle_HRO_TYPE-C-31-M-12"
 			(at 55.88 63.5 0)
 			(hide yes)
@@
 			)
 		)
-		(property "Footprint" ""
+		(property "Footprint" "Capacitor_SMD:C_0805_2012Metric"
 			(at 140.6652 55.88 0)
 			(hide yes)
