File: hardware/numpad/03_matrix.kicad_sch (KiCad schematic)
At the start: 0 parts

Commit message: matrix sheet, encoder, root hierarchy wired
Parts:
- added D1, D10, D11, D12, D13, D14, D15, D16, D17, D18, D2, D3, D4, D5, D6, D7, D8, D9: 1N4148W, Diode_SMD:D_SOD-123, symbol Diode:1N4148W
- added MX1: NUM, PCM_marbastlib-mx:SW_MX_HS_CPG151101S11_1u, symbol marbastlib-mx:MX_SW_HS_CPG151101S11
- added MX10: 5, PCM_marbastlib-mx:SW_MX_HS_CPG151101S11_1u, symbol marbastlib-mx:MX_SW_HS_CPG151101S11
- added MX11: 6, PCM_marbastlib-mx:SW_MX_HS_CPG151101S11_1u, symbol marbastlib-mx:MX_SW_HS_CPG151101S11
- added MX12: 1, PCM_marbastlib-mx:SW_MX_HS_CPG151101S11_1u, symbol marbastlib-mx:MX_SW_HS_CPG151101S11
- added MX13: 2, PCM_marbastlib-mx:SW_MX_HS_CPG151101S11_1u, symbol marbastlib-mx:MX_SW_HS_CPG151101S11
- added MX14: 3, PCM_marbastlib-mx:SW_MX_HS_CPG151101S11_1u, symbol marbastlib-mx:MX_SW_HS_CPG151101S11
- added MX15: 0, PCM_marbastlib-mx:SW_MX_HS_CPG151101S11_1u, symbol marbastlib-mx:MX_SW_HS_CPG151101S11
- added MX16: PERIOD, PCM_marbastlib-mx:SW_MX_HS_CPG151101S11_1u, symbol marbastlib-mx:MX_SW_HS_CPG151101S11
- added MX17: ENTER, PCM_marbastlib-mx:SW_MX_HS_CPG151101S11_1u, symbol marbastlib-mx:MX_SW_HS_CPG151101S11
- added MX2: DIV, PCM_marbastlib-mx:SW_MX_HS_CPG151101S11_1u, symbol marbastlib-mx:MX_SW_HS_CPG151101S11
- added MX3: MULT, PCM_marbastlib-mx:SW_MX_HS_CPG151101S11_1u, symbol marbastlib-mx:MX_SW_HS_CPG151101S11
- added MX4: MIN, PCM_marbastlib-mx:SW_MX_HS_CPG151101S11_1u, symbol marbastlib-mx:MX_SW_HS_CPG151101S11
- added MX5: 7, PCM_marbastlib-mx:SW_MX_HS_CPG151101S11_1u, symbol marbastlib-mx:MX_SW_HS_CPG151101S11
- added MX6: 8, PCM_marbastlib-mx:SW_MX_HS_CPG151101S11_1u, symbol marbastlib-mx:MX_SW_HS_CPG151101S11
- added MX7: 9, PCM_marbastlib-mx:SW_MX_HS_CPG151101S11_1u, symbol marbastlib-mx:MX_SW_HS_CPG151101S11
- added MX8: PLUS, PCM_marbastlib-mx:SW_MX_HS_CPG151101S11_1u, symbol marbastlib-mx:MX_SW_HS_CPG151101S11
- added MX9: 4, PCM_marbastlib-mx:SW_MX_HS_CPG151101S11_1u, symbol marbastlib-mx:MX_SW_HS_CPG151101S11
- added SW3: RotaryEncoder_Switch, symbol Device:RotaryEncoder_Switch
Connections:
- new net: D4.2 (A), MX4.1
- new net: D11.2 (A), MX11.1
- new net: D2.2 (A), MX2.1
- new net: D16.2 (A), MX16.1
- new net: D6.2 (A), MX6.1
- new net: D7.2 (A), MX7.1
- new net: D8.2 (A), MX8.1
- new net: D17.2 (A), MX17.1
- new net: D10.2 (A), MX10.1
- new net: D18.2 (A), SW3.S2
- new net: D3.2 (A), MX3.1
- new net: D1.2 (A), MX1.1
- new net: D5.2 (A), MX5.1
- new net: D14.2 (A), MX14.1
- new net: D9.2 (A), MX9.1
- new net: D12.2 (A), MX12.1
- new net: D13.2 (A), MX13.1
- new net: D15.2 (A), MX15.1
- new net COL0: MX1.2, MX12.2, MX15.2, MX5.2, MX9.2
- new net COL1: MX10.2, MX13.2, MX2.2, MX6.2
- new net COL2: MX11.2, MX14.2, MX16.2, MX3.2, MX7.2
- new net COL3: MX17.2, MX4.2, MX8.2, SW3.S1
- new net ENC_A: SW3.A
- new net ENC_B: SW3.B
- new net GND: SW3.C
- new net ROW0: D1.1 (K), D2.1 (K), D3.1 (K), D4.1 (K)
- new net ROW1: D5.1 (K), D6.1 (K), D7.1 (K), D8.1 (K)
- new net ROW2: D10.1 (K), D11.1 (K), D18.1 (K), D9.1 (K)
- new net ROW3: D12.1 (K), D13.1 (K), D14.1 (K)
- new net ROW4: D15.1 (K), D16.1 (K), D17.1 (K)

Commit message: Format cleanup, titles
Other:
- title: (none) -> Switch Matrix
- moved on the sheet: D1, D10, D11, D12, D13, D14, D15, D16, D17, D18, D2, D3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

Commit message: footprints set
Parts:
- SW3: footprint (none) -> Rotary_Encoder:RotaryEncoder_Alps_EC11E-Switch_Vertical_H20mm
Changed lines of the file:
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@@
 			)
 		)
-		(property "Footprint" ""
+		(property "Footprint" "Rotary_Encoder:RotaryEncoder_Alps_EC11E-Switch_Vertical_H20mm"
 			(at 176.53 94.234 0)
 			(hide yes)
