File: hardware/numpad/05_ui.kicad_sch (KiCad schematic)
At the start: 0 parts

Commit message: LCD header with I2C level shifting, schematic complete
Parts:
- added J3: Conn_01x04, symbol Connector_Generic:Conn_01x04
- added Q1, Q2: BSS138, Package_TO_SOT_SMD:SOT-23, symbol Transistor_FET:BSS138
- added R10, R11: 4k7, symbol Device:R
Connections:
- new net: J3.3 (Pin_3), Q1.3 (D)
- new net: J3.4 (Pin_4), Q2.3 (D)
- new net +3V3: Q1.1 (G), Q2.1 (G), R10.1, R11.1
- new net +5V: J3.2 (Pin_2)
- new net GND: J3.1 (Pin_1)
- new net I2C_SCL: Q2.2 (S), R11.2
- new net I2C_SDA: Q1.2 (S), R10.2
Other:
- note added: "high-side I2C pullups on LCD backpack module"

Commit message: Format cleanup, titles
Other:
- title: (none) -> LCD I2C Connectors
- moved on the sheet: J3, Q1, Q2, R10, R11

Commit message: footprints set
Parts:
- J3: footprint (none) -> Connector_PinHeader_2.54mm:PinHeader_1x04_P2.54mm_Vertical
- R10, R11: footprint (none) -> Resistor_SMD:R_0603_1608Metric
Changed lines of the file:
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@@
 			)
 		)
-		(property "Footprint" ""
+		(property "Footprint" "Resistor_SMD:R_0603_1608Metric"
 			(at 74.422 64.77 90)
 			(hide yes)
@@
 			)
 		)
-		(property "Footprint" ""
+		(property "Footprint" "Resistor_SMD:R_0603_1608Metric"
 			(at 96.012 62.23 90)
 			(hide yes)
@@
 			)
 		)
-		(property "Footprint" ""
+		(property "Footprint" "Connector_PinHeader_2.54mm:PinHeader_1x04_P2.54mm_Vertical"
 			(at 123.19 63.5 0)
 			(hide yes)
